File: kicad/LPC55Sxx.sch (KiCad schematic (older format))
At the start: 7 parts, among them U1 LPC55S28JEV98K

Commit message: new nfc chip layout
Connections:
- net NFC_GPIO: now reaches U1.L12 (PIO0_0/ACMP0_A/FC3_SCK/CTIMER0_MAT0/SCT0_GPI0/SD1_CARD_INT_N/SEC_PIO0_0)
Changed lines of the file:
@@
 Text HLabel 8950 2800 2    50   Input ~ 0
 SENSE3
-Text HLabel 8950 2950 2    50   Input ~ 0
-CHARGE1
-Text HLabel 8950 3050 2    50   Input ~ 0
-CHARGE2
-Text HLabel 8950 3150 2    50   Input ~ 0
-CHARGE3
 Text Notes 8300 2550 0    50   ~ 0
 Support 3 capacitive touch buttons.\nUses RC acquisition principle.  \nSee ST AN2927.
@@
 Text Label 6500 3200 0    50   ~ 0
 SENSE2
-Wire Wire Line
-	6450 4100 6200 4100
 Text Notes 6850 3200 0    50   ~ 0
 COMP input B
@@
 Wire Wire Line
 	10500 4950 10650 4950
+Text HLabel 8900 2100 2    50   Input ~ 0
+NFC_GPIO
+Text Label 6450 4150 0    50   ~ 0
+NFC_GPIO
+Wire Wire Line
+	6450 4150 6350 4150
+Wire Wire Line
+	6350 4150 6350 4100
+Wire Wire Line
+	6350 4100 6200 4100
+Text HLabel 8950 3150 2    50   Input ~ 0
+CHARGE3
+Text HLabel 8950 3050 2    50   Input ~ 0
+CHARGE2
+Text HLabel 8950 2950 2    50   Input ~ 0
+CHARGE1
 $EndSCHEMATC
