File: kicad/solo.sch (KiCad schematic (older format))
At the start: 26 parts, among them T1 TLV742p

Commit message: new nfc chip layout
Parts:
- removed N1: AS3953-CSP, solo:AS3953_CSP, symbol solo:AS3953-CSP
- added N1: FM11NC08I, solo:MLPD3X3, symbol solo:AMS3956
Connections:
- wire segments 187 -> 196
- no-connect marks 1 -> 0
Other:
- moved on the sheet: AE1, CX1, CY1
Changed lines of the file:
@@
 F26 "FLASH_POWER" I L 6700 4700 50
 F27 "FLASH_SS" I L 6700 4550 50
+F28 "NFC_GPIO" I L 6700 3550 50
 $EndSheet
 $Comp
@@
 Text Label 8650 3900 0    50   ~ 0
 nRESET
-NoConn ~ 4550 3650
 $Comp
 L power:GNDREF #PWR03
@@
 Wire Wire Line
 	6250 2800 6700 2800
-$Comp
-L Device:Antenna_Loop AE1
-U 1 1 5DE36C4B
-P 1500 4050
-F 0 "AE1" V 1867 4018 50  0000 C CNN
-F 1 "Antenna_Loop" V 1776 4018 50  0000 C CNN
-F 2 "" H 1500 4050 50  0001 C CNN
-F 3 "~" H 1500 4050 50  0001 C CNN
-	1    1500 4050
-	0    -1   -1   0
-$EndComp
 $Comp
 L solo:TLV742p T1
@@
 	5650 3200 6700 3200
 Wire Wire Line
-	1750 4100 1750 4050
-Wire Wire Line
-	1750 4050 1700 4050
+	1550 4100 1550 4050
 Wire Wire Line
 	3550 3950 3250 3950
 Wire Wire Line
-	3250 3950 3250 3850
-Wire Wire Line
-	2500 3850 2300 3850
-Wire Wire Line
-	2300 3850 2300 3950
-Connection ~ 2500 3850
-Wire Wire Line
-	1700 3950 2300 3950
+	2300 3850 2100 3850
+Wire Wire Line
+	2100 3850 2100 3950
+Connection ~ 2300 3850
 Wire Wire Line
 	3550 4100 3250 4100
@@
 	3250 4100 3250 4150
 Wire Wire Line
-	2500 4150 2300 4150
-Wire Wire Line
-	2300 4150 2300 4100
-Connection ~ 2500 4150
-Wire Wire Line
-	1750 4100 2300 4100
+	2300 4150 2100 4150
+Wire Wire Line
+	2100 4150 2100 4100
+Connection ~ 2300 4150
+Wire Wire Line
+	1550 4100 2100 4100
 Wire Wire Line
 	9450 1600 9450 1550
@@
 Text HLabel 9000 1550 0    50   Input ~ 0
 CAP3
-Text HLabel 2050 3950 1    50   Input ~ 0
+Text HLabel 1850 3950 1    50   Input ~ 0
 NFC+
-Text HLabel 2050 4100 3    50   Input ~ 0
+Text HLabel 1850 4100 3    50   Input ~ 0
 NFC-
 $Comp
@@
 L Device:C CX1
 U 1 1 5DF3E27E
-P 2500 4000
-F 0 "CX1" H 2615 4046 50  0000 L CNN
-F 1 "DNP" H 2615 3955 50  0000 L CNN
-F 2 "solo:0201_C" H 2538 3850 50  0001 C CNN
-F 3 "~" H 2500 4000 50  0001 C CNN
-F 4 "" H 2500 4000 50  0001 C CNN "Manufacturer"
-F 5 "" H 2500 4000 50  0001 C CNN "Description"
-F 6 "" H 2500 4000 50  0001 C CNN "MPN"
-F 7 "2" H 2500 4000 50  0001 C CNN "Pins"
-F 8 "0201" H 2500 4000 50  0001 C CNN "Package"
-	1    2500 4000
-	1    0    0    -1
-$EndComp
-Wire Wire Line
-	2500 3850 2900 3850
-Wire Wire Line
-	2500 4150 2900 4150
+P 2300 4000
+F 0 "CX1" H 2415 4046 50  0000 L CNN
+F 1 "DNP" H 2415 3955 50  0000 L CNN
+F 2 "solo:0201_C" H 2338 3850 50  0001 C CNN
+F 3 "~" H 2300 4000 50  0001 C CNN
+F 4 "" H 2300 4000 50  0001 C CNN "Manufacturer"
+F 5 "" H 2300 4000 50  0001 C CNN "Description"
+F 6 "" H 2300 4000 50  0001 C CNN "MPN"
+F 7 "2" H 2300 4000 50  0001 C CNN "Pins"
+F 8 "0201" H 2300 4000 50  0001 C CNN "Package"
+	1    2300 4000
+	1    0    0    -1
+$EndComp
+Wire Wire Line
+	2300 3850 2700 3850
+Wire Wire Line
+	2300 4150 2700 4150
 $Comp
 L Device:C CY1
 U 1 1 5DF47EDF
-P 2900 4000
-F 0 "CY1" H 3015 4046 50  0000 L CNN
-F 1 "DNP" H 3015 3955 50  0000 L CNN
-F 2 "solo:0201_C" H 2938 3850 50  0001 C CNN
-F 3 "~" H 2900 4000 50  0001 C CNN
-F 4 "" H 2900 4000 50  0001 C CNN "Manufacturer"
-F 5 "" H 2900 4000 50  0001 C CNN "Description"
-F 6 "" H 2900 4000 50  0001 C CNN "MPN"
-F 7 "2" H 2900 4000 50  0001 C CNN "Pins"
-F 8 "0201" H 2900 4000 50  0001 C CNN "Package"
-	1    2900 4000
-	1    0    0    -1
-$EndComp
-Connection ~ 2900 3850
-Wire Wire Line
-	2900 3850 3250 3850
-Connection ~ 2900 4150
-Wire Wire Line
-	2900 4150 3250 4150
+P 2700 4000
+F 0 "CY1" H 2815 4046 50  0000 L CNN
+F 1 "DNP" H 2815 3955 50  0000 L CNN
+F 2 "solo:0201_C" H 2738 3850 50  0001 C CNN
+F 3 "~" H 2700 4000 50  0001 C CNN
+F 4 "" H 2700 4000 50  0001 C CNN "Manufacturer"
+F 5 "" H 2700 4000 50  0001 C CNN "Description"
+F 6 "" H 2700 4000 50  0001 C CNN "MPN"
+F 7 "2" H 2700 4000 50  0001 C CNN "Pins"
+F 8 "0201" H 2700 4000 50  0001 C CNN "Package"
+	1    2700 4000
+	1    0    0    -1
+$EndComp
+Connection ~ 2700 3850
+Connection ~ 2700 4150
+Wire Wire Line
+	2700 4150 3050 4150
 $Comp
 L Device:C C1
@@
 $EndComp
 $Comp
-L solo:AS3953-CSP N1
-U 1 1 5E160F94
-P 4450 4550
-F 0 "N1" H 4850 4615 50  0000 C CNN
-F 1 "AS3953-CSP" H 4850 4524 50  0000 C CNN
-F 2 "solo:AS3953_CSP" H 4950 4500 50  0001 C CNN
-F 3 "" H 4950 4500 50  0001 C CNN
-	1    4450 4550
+L power:GNDREF #PWR0113
+U 1 1 5E1F57F6
+P 3900 3100
+F 0 "#PWR0113" H 3900 2850 50  0001 C CNN
+F 1 "GNDREF" H 3905 2927 50  0000 C CNN
+F 2 "" H 3900 3100 50  0001 C CNN
+F 3 "" H 3900 3100 50  0001 C CNN
+	1    3900 3100
+	0    1    1    0
+$EndComp
+Wire Wire Line
+	4050 3400 4050 3100
+Wire Wire Line
+	4050 3100 3900 3100
+Wire Wire Line
+	6700 3550 5450 3550
+Wire Wire Line
+	5450 3550 5450 3650
+Wire Wire Line
+	5450 3650 4550 3650
+Wire Wire Line
+	1500 3950 2100 3950
+Wire Wire Line
+	1550 4050 1500 4050
+$Comp
+L Device:Antenna_Loop AE1
+U 1 1 5DE36C4B
+P 1300 4050
+F 0 "AE1" V 1667 4018 50  0000 C CNN
+F 1 "Antenna_Loop" V 1576 4018 50  0000 C CNN
+F 2 "" H 1300 4050 50  0001 C CNN
+F 3 "~" H 1300 4050 50  0001 C CNN
+	1    1300 4050
+	0    -1   -1   0
+$EndComp
+$Comp
+L solo:AMS3956 N1
+U 1 1 5E1F1BCD
+P 4450 4450
+F 0 "N1" H 4850 4523 50  0000 C CNN
+F 1 "FM11NC08I" H 4850 4614 50  0000 C CNN
+F 2 "solo:MLPD3X3" H 5100 4600 50  0001 C CNN
+F 3 "" H 5100 4600 50  0001 C CNN
+	1    4450 4450
 	-1   0    0    1
 $EndComp
+Wire Wire Line
+	3200 3850 3200 4150
+Wire Wire Line
+	3200 4150 3250 4150
+Wire Wire Line
+	2700 3850 3200 3850
+Wire Wire Line
+	3050 4150 3050 3750
+Wire Wire Line
+	3050 3750 3250 3750
+Wire Wire Line
+	3250 3750 3250 3950
 $EndSCHEMATC
